File: CalliopeGamePad.kicad_sch (KiCad schematic)
At the start: 26 parts, among them J1 Conn_02x15_Odd_Even, J2 Conn_01x04, U1 SW_MEC_5E, U2 SW_MEC_5E, U3 SW_MEC_5E, U4 SW_MEC_5E, U5 SW_MEC_5E, U6 SW_MEC_5E, U7 SW_MEC_5E, U8 SW_MEC_5E

Commit message: UPDATE socket footprint in kicad_sch
Parts:
- J1: footprint Connector_PinSocket_2.54mm:PinSocket_2x15_P2.54mm_Vertical -> Connector_PinHeader_2.54mm:PinHeader_2x15_P2.54mm_Vertical
Changed lines of the file:
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@@
 			)
 		)
-		(property "Footprint" "Connector_PinSocket_2.54mm:PinSocket_2x15_P2.54mm_Vertical"
+		(property "Footprint" "Connector_PinHeader_2.54mm:PinHeader_2x15_P2.54mm_Vertical"
 			(at 149.86 53.34 0)
 			(effects
